File: 1800muente FAIL.sch (KiCad schematic (older format))
At the start: 163 parts, among them K1 MX-1U, K10 MX-1U, K11 MX-1U, K12 MX-1U, K13 MX-1U, K14 MX-1U, K15 MX-1U, K16 MX-1U, K17 MX-1U, K18 MX-1U, K19 MX-1U, K2 MX-1U, K20 MX-1U, K21 MX-1U, K22 MX-1U, K23 MX-1U, K24 MX-1U, K25 MX-1U, K26 MX-1U, K27 MX-1U, K28 MX-1U, K29 MX-1U, K3 MX-1U, K30 MX-1U, K31 MX-1U, K32 MX-1U, K33 MX-1U, K34 MX-1U, K35 MX-1U, K36 MX-1U, K37 MX-1U, K38 MX-1U, K39 MX-1U, K4 MX-1U, K40 MX-1U, K41 MX-1U, K42 MX-1U, K43 MX-1U, K44 MX-1U, K45 MX-1U, K46 MX-1U, K47 MX-1U, K48 MX-1U, K49 MX-1U, K5 MX-1U, K50 MX-1U, K51 MX-1U, K52 MX-1U, K53 MX-1U, K54 MX-1U, K55 MX-1U, K56 MX-1U, K57 MX-1U, K58 MX-1U, K59 MX-1U, K6 MX-1U, K60 MX-1U, K61 MX-1U, K62 MX-1U, K63 MX-1U, K64 MX-1U, K65 MX-1U, K66 MX-1U, K67 MX-1U, K68 MX-1U, K69 MX-1U, K7 MX-1U, K70 MX-1U, K71 MX-1U, K72 MX-1U, K73 MX-1U, K74 MX-1U, K75 MX-1U, K76 MX-1U, K77 MX-1U, K78 MX-1U, K79 MX-1U, K8 MX-1U, K80 MX-1U, K81 MX-1U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

Commit message: changing layout
Parts:
- added D75, D83: D_Small, symbol Device:D_Small
- added K75, K83: MX-1U, symbol MX_Alps_Hybrids:MX-1U
- renumbered D15 to D10, D10 to D11, D11 to D12, D12 to D13, D13 to D14, D14 to D15, D24 to D19, D19 to D20, D20 to D21, D21 to D22, D22 to D23, D23 to D24, D33 to D28, D28 to D29, D29 to D30, D30 to D31, D31 to D32, D32 to D33, D42 to D37, D37 to D38, D38 to D39, D39 to D40, D40 to D41, D41 to D42, D80 to D46, D46 to D47, D47 to D48, D48 to D49, D49 to D50, D50 to D51, D51 to D52, D52 to D53, D53 to D54, D54 to D55, D62 to D56, D55 to D57, D56 to D58, D57 to D59, D58 to D60, D59 to D61, D60 to D62, D61 to D63, D63 to D64, D78 to D65, D64 to D66, D65 to D67, D66 to D68, D67 to D69, D68 to D70, D69 to D71, D70 to D72, D71 to D73, D72 to D74, D73 to D76, D74 to D77, D75 to D78, D76 to D79, D77 to D80, D79 to D81, D81 to D82, K15 to K10, K10 to K11, K11 to K12, K12 to K13, K13 to K14, K14 to K15, K24 to K19, K19 to K20, K20 to K21, K21 to K22, K22 to K23, K23 to K24, K33 to K28, K28 to K29, K29 to K30, K30 to K31, K31 to K32, K32 to K33, K42 to K37, K37 to K38, K38 to K39, K39 to K40, K40 to K41, K41 to K42, K80 to K46, K46 to K47, K47 to K48, K48 to K49, K49 to K50, K50 to K51, K51 to K52, K52 to K53, K53 to K54, K54 to K55, K62 to K56, K55 to K57, K56 to K58, K57 to K59, K58 to K60, K59 to K61, K60 to K62, K61 to K63, K63 to K64, K78 to K65, K64 to K66, K65 to K67, K66 to K68, K67 to K69, K68 to K70, K69 to K71, K70 to K72, K71 to K73, K72 to K74, K73 to K76, K74 to K77, K75 to K78, K76 to K79, K77 to K80, K79 to K81, K81 to K82, U1 to U?
Connections:
- net col0: now also K10.1 (COL)
- net col1: now also K19.1 (COL); no longer K10.1 (COL)
- net col2: now also K28.1 (COL); no longer K19.1 (COL)
- net col3: now also K37.1 (COL); no longer K28.1 (COL)
- net col4: now also K46.1 (COL); no longer K37.1 (COL)
- net col5: now also K56.1 (COL)
- net col6: now also K65.1 (COL); no longer K56.1 (COL)
- net col7: now also K75.1 (COL)
- net col8: now also K83.1 (COL); no longer K46.1 (COL), K65.1 (COL), U?.12 (9/PB5)
- net row5: no longer D10.1 (K), D19.1 (K), D28.1 (K), D37.1 (K), D65.1 (K)
- net row7: no longer D46.1 (K), D56.1 (K)
- new net: D75.2 (A), K75.2 (ROW)
- new net: D83.2 (A), K83.2 (ROW)
- new net row9: D10.1 (K), D19.1 (K), D28.1 (K), D37.1 (K), D46.1 (K), D56.1 (K), D65.1 (K), D75.1 (K), D83.1 (K), U?.12 (9/PB5)
Other:
- moved on the sheet: D10, D19, D28, D37, D46, D56, D65, K10, K19, K28, K37, K46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
