File: 1800muente.kicad_pcb (KiCad board)
At the start: 2 copper layers, 163 parts, among them K1 MX-1U, K10 MX-1U, K11 MX-1U, K12 MX-1U, K13 MX-1U, K14 MX-1U, K15 MX-1U, K16 MX-1U, K17 MX-1U, K18 MX-1U, K19 MX-1U, K2 MX-1U, K20 MX-1U, K21 MX-1U, K22 MX-1U, K23 MX-1U, K24 MX-1U, K25 MX-1U, K26 MX-1U, K27 MX-1U, K28 MX-1U, K29 MX-1U, K3 MX-1U, K30 MX-1U, K31 MX-1U, K32 MX-1U, K33 MX-1U, K34 MX-1U, K35 MX-1U, K36 MX-1U, K37 MX-1U, K38 MX-1U, K39 MX-1U, K4 MX-1U, K40 MX-1U, K41 MX-1U, K42 MX-1U, K43 MX-1U, K44 MX-1U, K45 MX-1U, K46 MX-1U, K47 MX-1U, K48 MX-1U, K49 MX-1U, K5 MX-1U, K50 MX-1U, K51 MX-1U, K52 MX-1U, K53 MX-1U, K54 MX-1U, K55 MX-1U, K56 MX-1U, K57 MX-1U, K58 MX-1U, K59 MX-1U, K6 MX-1U, K60 MX-1U, K61 MX-1U, K62 MX-1U, K63 MX-1U, K64 MX-1U, K65 MX-1U, K66 MX-1U, K67 MX-1U, K68 MX-1U, K69 MX-1U, K7 MX-1U, K70 MX-1U, K71 MX-1U, K72 MX-1U, K73 MX-1U, K74 MX-1U, K75 MX-1U, K76 MX-1U, K77 MX-1U, K78 MX-1U, K79 MX-1U, K8 MX-1U, K80 MX-1U, K81 MX-1U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

Commit message: aligning switches
Parts:
- K61: footprint MX_Alps_Hybrid:MXOnly-2U-NoLED -> MX_Alps_Hybrid:MXOnly-ISO
- moved K7 618.4 mm to (64.5, 120.6)
- moved K1 608.5 mm to (35.9, 101.6)
- moved K16 596.1 mm to (93.1, 101.6)
- moved K8 594.2 mm to (69.2, 139.7)
- moved K20 593.9 mm to (112.1, 101.6)
- moved K9 579.1 mm to (59.7, 158.7)
- moved K17 563.2 mm to (102.6, 120.6)
- moved K25 556.1 mm to (140.7, 120.6)
- moved K18 539.1 mm to (107.3, 139.7)
- moved K13 536.8 mm to (88.3, 139.7)
- moved K19 524.2 mm to (97.8, 158.7)
- moved K23 518.6 mm to (116.9, 158.7)
- moved K11 518.1 mm to (74.0, 101.6)
- moved K12 516.9 mm to (83.5, 120.6)
- moved K6 509.1 mm to (55.0, 101.6)
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
Commit message: brb
Parts:
- added J1: Conn_01x04, Connector_PinSocket_2.54mm:PinSocket_1x04_P2.54mm_Vertical, F.Cu at (53.1, 116.2)
- added R1: 5.1k, Keebio-Parts:Resistor, F.Cu at (54.2, 136.5)
- added R2: 5.1k, Keebio-Parts:Resistor, F.Cu at (57.1, 136.5)
- added USB1: HRO-TYPE-C-31-M-12, Type-C:HRO-TYPE-C-31-M-12-HandSoldering, B.Cu at (45.5, 88.3)
- K3: footprint MX_Alps_Hybrid:MX-1.75U-NoLED -> MX_Alps_Hybrid:MXOnly-1.75U-NoLED
- moved D4 661.1 mm to (38.3, 166.4)
- moved D5 651.5 mm to (38.3, 185.4)
- moved D14 620.9 mm to (78.8, 166.4)
- moved D1 618.5 mm to (35.9, 109.2)
- moved D19 613.0 mm to (97.8, 166.4)
- moved D8 604.2 mm to (69.2, 147.3)
- moved D10 601.6 mm to (62.1, 185.4)
- moved D9 599.9 mm to (59.7, 166.4)
- moved D2 592.8 mm to (40.7, 128.3)
- moved D18 591.6 mm to (107.3, 147.3)
- moved D15 588.6 mm to (85.9, 185.4)
- moved D7 586.8 mm to (64.5, 128.3)
- moved D16 581.7 mm to (93.1, 107.2)
- moved D6 580.8 mm to (55.0, 109.2)
- moved D11 579.9 mm to (74.0, 107.2)
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Routing:
- net col6: track 0.00 -> 208.6 mm
- net col8: track 0.00 -> 198.9 mm
- net col0: track 0.00 -> 178.3 mm
- net col7: track 0.00 -> 176.7 mm
- net col1: track 0.00 -> 94.1 mm
- net row4: track 0.00 -> 39.1 mm
- net Net-(D59-Pad2): track 0.00 -> 13.9 mm
- net Net-(D79-Pad2): track 0.00 -> 13.9 mm
- net Net-(D60-Pad2): track 0.00 -> 13.9 mm
- net Net-(D55-Pad2): track 0.00 -> 13.9 mm
- net Net-(D81-Pad2): track 0.00 -> 13.9 mm
- net Net-(D80-Pad2): track 0.00 -> 13.9 mm
- net Net-(D44-Pad2): track 0.00 -> 13.9 mm
- net Net-(D36-Pad2): track 0.00 -> 13.9 mm
- net Net-(D23-Pad2): track 0.00 -> 13.9 mm
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- added copper zone on B.Cu, net GND
- added copper zone on F.Cu, net GND
Other:
- board outline added: 379.5 x 108 mm

Commit message: gerbers ready
Routing:
- net row0: track 0.00 -> 561.1 mm, vias 0 -> 1
- net row5: track 0.00 -> 504.1 mm
- net row4: track 39.1 -> 532.9 mm
- net row8: track 0.00 -> 481.6 mm
- net row3: track 0.00 -> 401.7 mm
- net row1: track 0.00 -> 396.6 mm
- net row6: track 0.00 -> 382.8 mm
- net row7: track 0.00 -> 375.5 mm
- net row2: track 0.00 -> 371.9 mm, vias 0 -> 1
- net col5: track 0.00 -> 304.8 mm
- net col8: track 198.9 -> 482.8 mm
- net col4: track 0.00 -> 247.0 mm
- net col7: track 176.7 -> 409.2 mm
- net col3: track 0.00 -> 214.7 mm
- net col2: track 0.00 -> 185.0 mm
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- removed copper zone on B.Cu, net GND
- removed copper zone on F.Cu, net GND

Commit message: m2 mounting holes
Parts:
- added M2_1: MountingHole_2.2mm_M2, MountingHole:MountingHole_2.2mm_M2, F.Cu at (306.0, 194.1)
- added M2_1: MountingHole_2.2mm_M2, MountingHole:MountingHole_2.2mm_M2, F.Cu at (24.4, 194.1)
- added M2_1: MountingHole_2.2mm_M2, MountingHole:MountingHole_2.2mm_M2, F.Cu at (24.4, 142.1)
- added M2_1: MountingHole_2.2mm_M2, MountingHole:MountingHole_2.2mm_M2, F.Cu at (24.4, 90.1)
- added M2_1: MountingHole_2.2mm_M2, MountingHole:MountingHole_2.2mm_M2, F.Cu at (212.1, 194.1)
- added M2_1: MountingHole_2.2mm_M2, MountingHole:MountingHole_2.2mm_M2, F.Cu at (118.6, 194.1)
- added M2_1: MountingHole_2.2mm_M2, MountingHole:MountingHole_2.2mm_M2, F.Cu at (212.1, 90.1)
- added M2_1: MountingHole_2.2mm_M2, MountingHole:MountingHole_2.2mm_M2, F.Cu at (306.0, 90.1)
- added M2_1: MountingHole_2.2mm_M2, MountingHole:MountingHole_2.2mm_M2, F.Cu at (118.3, 90.1)
- added M2_1: MountingHole_2.2mm_M2, MountingHole:MountingHole_2.2mm_M2, F.Cu at (399.8, 90.1)
- added M2_1: MountingHole_2.2mm_M2, MountingHole:MountingHole_2.2mm_M2, F.Cu at (399.8, 142.1)
- added M2_1: MountingHole_2.2mm_M2, MountingHole:MountingHole_2.2mm_M2, F.Cu at (399.8, 194.1)
Other:
- outline, holes or cut-outs redrawn

Commit message: adding iso layout
Parts:
- removed the M2_1 at (24.4, 194.1)
- removed the M2_1 at (24.4, 142.1)
- added K4_2: MX-1U, MX_Alps_Hybrid:MXOnly-2.25U-NoLED, F.Cu at (47.8, 158.7)
- added K57_2: MX-1U, MX_Alps_Hybrid:MXOnly-1.5U-NoLED, F.Cu at (297.8, 120.6)
- added K61_2: MX-1U, MX_Alps_Hybrid:MXOnly-2.25U-NoLED, F.Cu at (290.7, 139.7)
- added M2_6: MountingHole_2.2mm_M2, MountingHole:MountingHole_2.2mm_M2, F.Cu at (24.4, 142.1)
- added M2_8: MountingHole_2.2mm_M2, MountingHole:MountingHole_2.2mm_M2, F.Cu at (24.4, 194.1)
- moved D61 15.1 mm to (313.3, 130.2), turned to 90 degrees
- moved D57 11.8 mm to (269.9, 139.6), turned to 90 degrees
- moved D9 7.45 mm to (67.2, 166.3)
- moved D4 5.40 mm to (43.7, 166.3)
- renumbered M2_1 to M2_10, M2_1 to M2_11, M2_1 to M2_12, M2_1 to M2_2, M2_1 to M2_3, M2_1 to M2_4, M2_1 to M2_5, M2_1 to M2_7, M2_1 to M2_9
Routing:
- net row0: track 561.1 -> 0.00 mm, vias 1 -> 0
- net row4: track 532.9 -> 0.00 mm
- net row5: track 504.1 -> 0.00 mm
- net col8: track 482.8 -> 0.00 mm
- net row8: track 481.6 -> 0.00 mm
- net col7: track 409.2 -> 0.00 mm
- net row3: track 401.7 -> 0.00 mm
- net row1: track 396.6 -> 0.00 mm
- net row6: track 382.8 -> 0.00 mm
- net row7: track 375.5 -> 0.00 mm
- net row2: track 371.9 -> 0.00 mm, vias 1 -> 0
- net col6: track 371.8 -> 0.00 mm
- net col5: track 304.8 -> 0.00 mm
- net col4: track 247.0 -> 0.00 mm
- net col3: track 214.7 -> 0.00 mm
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
Commit message: iso support
Routing:
- net row0: track 0.00 -> 561.1 mm
- net row4: track 0.00 -> 557.1 mm
- net row5: track 0.00 -> 523.2 mm
- net row8: track 0.00 -> 451.8 mm
- net row1: track 0.00 -> 429.6 mm, vias 0 -> 1
- net col8: track 0.00 -> 426.3 mm
- net row3: track 0.00 -> 393.6 mm
- net col7: track 0.00 -> 389.3 mm
- net row2: track 0.00 -> 380.8 mm
- net row6: track 0.00 -> 379.4 mm
- net row7: track 0.00 -> 364.2 mm
- net col6: track 0.00 -> 358.1 mm
- net col5: track 0.00 -> 295.9 mm
- net col4: track 0.00 -> 253.7 mm
- net col3: track 0.00 -> 220.5 mm
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
Commit message: fixed
Parts:
- moved D60 18.9 mm to (275.5, 102.4), turned to 90 degrees
- moved D4 16.2 mm to (29.3, 158.8), turned to 90 degrees
- moved D32 12.8 mm to (146.9, 177.9), turned to 90 degrees
- moved D12 1.00 mm to (82.9, 131.7)
- moved D17 1.00 mm to (101.9, 131.7)
- turned K57_2 to 0 degrees
Routing:
- net row0: track 561.1 -> 0.00 mm
- net row4: track 557.1 -> 0.00 mm
- net row5: track 523.2 -> 0.00 mm
- net row8: track 451.8 -> 0.00 mm
- net row1: track 429.6 -> 0.00 mm, vias 1 -> 0
- net col8: track 426.3 -> 0.00 mm
- net row3: track 393.6 -> 0.00 mm
- net col7: track 389.3 -> 0.00 mm
- net row2: track 380.8 -> 0.00 mm
- net row6: track 379.4 -> 0.00 mm
- net row7: track 364.2 -> 0.00 mm
- net col6: track 358.1 -> 0.00 mm
- net col5: track 295.9 -> 0.00 mm
- net col4: track 253.7 -> 0.00 mm
- net col3: track 220.5 -> 0.00 mm
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
Commit message: pcb design done
Parts:
- removed M2_1, M2_10, M2_11, M2_12, M2_2, M2_3, M2_4, M2_5, M2_6, M2_7, M2_8, M2_9: MountingHole_2.2mm_M2, MountingHole:MountingHole_2.2mm_M2
- moved D61 29.6 mm to (285.2, 120.7)
Other:
- board size 379.5 x 108 mm -> 371.5 x 104 mm
